Commit message: 增加雷达模型

File: rm_gimbal_description/urdf/rm_gimbal.urdf.xacro (robot description, xacro)
@@ -4,5 +4,5 @@
   <xacro:arg name="xyz" default="0.10 0 0.05" />
   <xacro:arg name="rpy" default="0 0 0" />
-  <xacro:arg name="lidar_xyz" default="0.0 -0.12 0.11" />
+  <xacro:arg name="lidar_xyz" default="0.0 -0.12 -0.11" />
   <xacro:arg name="lidar_rpy" default="0 0 0" />
   <link name="odom" />
@@ -13,5 +13,5 @@
     <child link="gimbal_link" />
   </joint>
-  <joint name="gimbal_yaw_joint" type="fixed">
+  <joint name="gimbal_yaw_joint" type="floating">
     <parent link="odom" />
     <child link="gimbal_yaw" />

Commit message: 优化代码

File: rm_gimbal_description/urdf/rm_gimbal.urdf.xacro (robot description, xacro)
@@ -35,4 +35,5 @@
     <parent link="gimbal_yaw" />
     <child link="front_mid360" />
+    <axis xyz="0 0 0" />
   </joint>
 </robot>
